File: elec/layout/default/expresslrs.kicad_pcb (KiCad board)
At the start: 2 copper layers, 225.7 x 100.8 mm, 0 parts

Commit message: initial layout
Parts:
- added C1: 10V 4.7uF X5R ±20% 0402 Multilayer Ceramic Capacitors MLCC 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, lib:C0402, F.Cu at (204.5, 101.4)
- added C10: 10V 470nF X5R ±10% 0402 Multilayer Ceramic Capacitors MLCC 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, lib:C0402, F.Cu at (220.7, 98.4)
- added C11: Multilayer Ceramic Capacitors MLCC - SMD/SMT 100nF 10V 0402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, lib:C0402, F.Cu at (219.6, 105.2)
- added C12: Multilayer Ceramic Capacitors MLCC - SMD/SMT 100nF 10V 0402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, lib:C0402, F.Cu at (216.5, 102.6)
- added C13: 50V 10nF X7R ±10% 0402 Multilayer Ceramic Capacitors MLCC -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, lib:C0402, F.Cu at (216.5, 103.5)
- added C14: 50V 10nF X7R ±10% 0402 Multilayer Ceramic Capacitors MLCC -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, lib:C0402, F.Cu at (221.8, 98.4)
- added C15: 50V 1pF C0G 0402 Multilayer Ceramic Capacitors MLCC - SMD/S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, lib:C0402, F.Cu at (223.4, 102.9)
- added C16: Multilayer Ceramic Capacitors MLCC - SMD/SMT 1.2pF 50V 0402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, lib:C0402, F.Cu at (224.0, 100.0)
- added C17: Multilayer Ceramic Capacitors MLCC - SMD/SMT 1.2pF 50V 0402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, lib:C0402, F.Cu at (226.9, 100.0)
- added C18: 50V 1pF C0G 0402 Multilayer Ceramic Capacitors MLCC - SMD/S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, lib:C0402, F.Cu at (225.5, 100.5)
- added C19: 50V 100pF C0G ±5% 0402 Multilayer Ceramic Capacitors MLCC -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, lib:C0402, F.Cu at (227.3, 101.4)
- added C2: Multilayer Ceramic Capacitors MLCC - SMD/SMT 100nF 10V 0402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, lib:C0402, F.Cu at (212.9, 104.0)
- added C3: Multilayer Ceramic Capacitors MLCC - SMD/SMT 1uF 6.3V 0402 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, lib:C0402, F.Cu at (204.5, 98.9)
- added C4: Multilayer Ceramic Capacitors MLCC - SMD/SMT 100nF 10V 0402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, lib:C0402, F.Cu at (212.9, 102.9)
- added C5: 50V 10nF X7R ±10% 0402 Multilayer Ceramic Capacitors MLCC -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, lib:C0402, F.Cu at (204.5, 97.9)
- added C6: 50V 13pF C0G ±2% 0402 Multilayer Ceramic Capacitors MLCC - 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, lib:C0402, F.Cu at (206.1, 105.6)
- added C7: 50V 13pF C0G ±2% 0402 Multilayer Ceramic Capacitors MLCC - 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, lib:C0402, F.Cu at (204.5, 102.4)
- added C8: Multilayer Ceramic Capacitors MLCC - SMD/SMT 10pF 50V 0402 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, lib:C0402, F.Cu at (220.7, 96.4)
- added C9: Multilayer Ceramic Capacitors MLCC - SMD/SMT 10pF 50V 0402 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, lib:C0402, F.Cu at (216.0, 96.9)
- added L1: , lib:L0402, F.Cu at (223.6, 101.4)
- added L2: , lib:L0402, F.Cu at (225.4, 101.4)
- added R1: Chip Resistor - Surface Mount 330Ohms ±5% 1/16W 0402 RoHS, lib:R0402, F.Cu at (208.4, 96.6)
- added R2: Chip Resistor - Surface Mount 10KOhms ±5% 1/16W 0402 RoHS, lib:R0402, F.Cu at (206.5, 96.5)
- added U1: , lib:UFQFPN-32_L5.0-W5.0-P0.50-TL-EP3.5, F.Cu at (208.7, 101.0)
- added U2: , lib:FC-135R_L3.2-W1.5, F.Cu at (204.3, 104.8)
- added U3: , lib:QFN-24_L4.0-W4.0-P0.50-BL-EP2.6, F.Cu at (219.9, 101.7)
- added U4: , lib:OSC-SMD_4P-L2.0-W1.6-BL, F.Cu at (218.3, 97.0)
- added U5: , lib:IPEX-SMD_BWIPX-1-001E, F.Cu at (229.8, 101.4)
- added U6: , lib:HDR-SMD_10P-P1.27-V-M-R2-C5-LS5.3, F.Cu at (212.6, 93.3)
Routing:
- net gnd: track 0.00 -> 24.1 mm, vias 0 -> 7
- net pb5: track 0.00 -> 12.7 mm, vias 0 -> 43
- net pc14_osc32_in: track 0.00 -> 12.5 mm
- net vcc: track 0.00 -> 10.5 mm, vias 0 -> 3
- net tx: track 0.00 -> 9.30 mm
- net vcc-3: track 0.00 -> 8.78 mm, vias 0 -> 2
- net pc15_osc32_out: track 0.00 -> 8.52 mm
- net tms: track 0.00 -> 6.10 mm
- net tdi: track 0.00 -> 5.23 mm, vias 0 -> 2
- net tck: track 0.00 -> 4.99 mm
- net io-2: track 0.00 -> 4.74 mm
- net tdo: track 0.00 -> 4.59 mm
- net rx: track 0.00 -> 3.13 mm
- net vcc-6: track 0.00 -> 2.86 mm
- net vcc-5: track 0.00 -> 2.86 mm
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